File: Placa/Placa tesis.sch (KiCad schematic (older format))
At the start: 78 parts, among them J1 Conn_01x03, J10 Conn_01x01, J11 USB_B_Micro, J12 Conn_01x01, J13 Conn_01x05, J14 Conn_01x08, J15 Conn_01x04, J2 Conn_01x04, J3 Conn_01x02, J4 Conn_01x03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

Commit message: actualizacion
Parts:
- C1: value 10n -> 1u
- C2, C4: value C -> 1u
- C3: value C -> 2.2n
- J11: symbol Placa-tesis-rescue:USB_B_Micro-Connector -> Placa-tesis-rescue:USB_B_Micro-Connector-Placa-tesis-rescue
- R1, R7: value R -> 10k
- R2: value R -> 4.7k
- R8: value R -> 1.5k
- SW1, SW2: renamed from SW?; footprint (none) -> Button_Switch_THT:SW_PUSH_6mm
- U2: symbol Placa-tesis-rescue:Nodemcuv_3-nodemcu-Placa-tesis-rescue -> Placa-tesis-rescue:Nodemcuv_3-nodemcu-Placa-tesis-rescue-Placa-tesis-rescue
- U4: symbol Placa-tesis-rescue:LM3464AMH_NOPB-LM3464AMH_NOPB-Placa-tesis-rescue -> Placa-tesis-rescue:LM3464AMH_NOPB-LM3464AMH_NOPB-Placa-tesis-rescue-Placa-tesis-rescue
- U9: symbol Placa-tesis-rescue:FT230XS-Interface_USB-Placa-tesis-rescue -> Placa-tesis-rescue:FT230XS-Interface_USB-Placa-tesis-rescue-Placa-tesis-rescue
- gave numbers to parts that had none: 4
Changed lines of the file:
@@
 $EndDescr
 $Comp
-L Placa-tesis-rescue:Nodemcuv_3-nodemcu-Placa-tesis-rescue U2
+L Placa-tesis-rescue:Nodemcuv_3-nodemcu-Placa-tesis-rescue-Placa-tesis-rescue U2
 U 1 1 5B848AAA
 P 12400 2300
@@
 P 4400 2550
 F 0 "R7" H 4470 2596 50  0000 L CNN
-F 1 "R" H 4470 2505 50  0000 L CNN
+F 1 "10k" H 4470 2505 50  0000 L CNN
 F 2 "Resistor_SMD:R_1206_3216Metric" V 4330 2550 50  0001 C CNN
 F 3 "~" H 4400 2550 50  0001 C CNN
@@
 P 4400 2950
 F 0 "R8" H 4470 2996 50  0000 L CNN
-F 1 "R" H 4470 2905 50  0000 L CNN
+F 1 "1.5k" H 4470 2905 50  0000 L CNN
 F 2 "Resistor_SMD:R_1206_3216Metric" V 4330 2950 50  0001 C CNN
 F 3 "~" H 4400 2950 50  0001 C CNN
@@
 P 850 1350
 F 0 "R1" H 920 1396 50  0000 L CNN
-F 1 "R" H 920 1305 50  0000 L CNN
+F 1 "10k" H 920 1305 50  0000 L CNN
 F 2 "Resistor_SMD:R_1206_3216Metric" V 780 1350 50  0001 C CNN
 F 3 "~" H 850 1350 50  0001 C CNN
@@
 P 850 1750
 F 0 "R2" H 920 1796 50  0000 L CNN
-F 1 "R" H 920 1705 50  0000 L CNN
+F 1 "4.7k" H 920 1705 50  0000 L CNN
 F 2 "Resistor_SMD:R_1206_3216Metric" V 780 1750 50  0001 C CNN
 F 3 "~" H 850 1750 50  0001 C CNN
@@
 P 850 2850
 F 0 "C1" H 968 2896 50  0000 L CNN
-F 1 "10n" H 968 2805 50  0000 L CNN
+F 1 "1u" H 968 2805 50  0000 L CNN
 F 2 "Capacitor_SMD:C_1206_3216Metric" H 888 2700 50  0001 C CNN
 F 3 "~" H 850 2850 50  0001 C CNN
@@
 P 1100 2000
 F 0 "C2" H 1218 2046 50  0000 L CNN
-F 1 "C" H 1218 1955 50  0000 L CNN
+F 1 "1u" H 1218 1955 50  0000 L CNN
 F 2 "Capacitor_SMD:C_1206_3216Metric" H 1138 1850 50  0001 C CNN
 F 3 "~" H 1100 2000 50  0001 C CNN
@@
 P 1250 2800
 F 0 "C3" H 1368 2846 50  0000 L CNN
-F 1 "C" H 1368 2755 50  0000 L CNN
+F 1 "2.2n" H 1368 2755 50  0000 L CNN
 F 2 "Capacitor_SMD:C_1206_3216Metric" H 1288 2650 50  0001 C CNN
 F 3 "~" H 1250 2800 50  0001 C CNN
@@
 	3750 4750 3850 4750
 $Comp
-L Placa-tesis-rescue:LM3464AMH_NOPB-LM3464AMH_NOPB-Placa-tesis-rescue U4
+L Placa-tesis-rescue:LM3464AMH_NOPB-LM3464AMH_NOPB-Placa-tesis-rescue-Placa-tesis-rescue U4
 U 1 1 5B8487B7
 P 2850 2250
@@
 P 4150 3150
 F 0 "C4" H 4268 3196 50  0000 L CNN
-F 1 "C" H 4268 3105 50  0000 L CNN
+F 1 "1u" H 4268 3105 50  0000 L CNN
 F 2 "Capacitor_SMD:C_1206_3216Metric" H 4188 3000 50  0001 C CNN
 F 3 "~" H 4150 3150 50  0001 C CNN
@@
 Vin
 $Comp
-L Placa-tesis-rescue:FT230XS-Interface_USB-Placa-tesis-rescue U9
+L Placa-tesis-rescue:FT230XS-Interface_USB-Placa-tesis-rescue-Placa-tesis-rescue U9
 U 1 1 5D99DAF0
 P 7250 9700
@@
 $EndComp
 $Comp
-L Placa-tesis-rescue:USB_B_Micro-Connector J11
+L Placa-tesis-rescue:USB_B_Micro-Connector-Placa-tesis-rescue J11
 U 1 1 5D99DB1A
 P 4850 9700
@@
 EN_esp
 $Comp
-L power:GND #PWR?
+L power:GND #PWR0101
 U 1 1 5F915214
 P 14800 4800
-F 0 "#PWR?" H 14800 4550 50  0001 C CNN
+F 0 "#PWR0101" H 14800 4550 50  0001 C CNN
 F 1 "GND" H 14805 4627 50  0000 C CNN
 F 2 "" H 14800 4800 50  0001 C CNN
@@
 V5
 $Comp
-L Device:R R?
+L Device:R R19
 U 1 1 5FA8A199
 P 15050 4700
-F 0 "R?" H 15120 4746 50  0000 L CNN
+F 0 "R19" H 15120 4746 50  0000 L CNN
 F 1 "10k" H 15120 4655 50  0000 L CNN
 F 2 "Resistor_SMD:R_1206_3216Metric" V 14980 4700 50  0001 C CNN
@@
 	14800 4700 14800 4800
 $Comp
-L Device:R R?
+L Device:R R18
 U 1 1 5FBC3573
 P 15050 4550
-F 0 "R?" H 15120 4596 50  0000 L CNN
+F 0 "R18" H 15120 4596 50  0000 L CNN
 F 1 "10k" H 15120 4505 50  0000 L CNN
 F 2 "Resistor_SMD:R_1206_3216Metric" V 14980 4550 50  0001 C CNN
@@
 $EndComp
 $Comp
-L Device:R R?
+L Device:R R17
 U 1 1 5FBC3969
 P 15050 4050
-F 0 "R?" H 15120 4096 50  0000 L CNN
+F 0 "R17" H 15120 4096 50  0000 L CNN
 F 1 "10k" H 15120 4005 50  0000 L CNN
 F 2 "Resistor_SMD:R_1206_3216Metric" V 14980 4050 50  0001 C CNN
@@
 $EndComp
 $Comp
-L Device:R R?
+L Device:R R16
 U 1 1 5FCBF9A8
 P 15050 3850
-F 0 "R?" H 15120 3896 50  0000 L CNN
+F 0 "R16" H 15120 3896 50  0000 L CNN
 F 1 "10k" H 15120 3805 50  0000 L CNN
 F 2 "Resistor_SMD:R_1206_3216Metric" V 14980 3850 50  0001 C CNN
@@
 	15200 4700 15550 4700
 $Comp
-L Switch:SW_Push SW?
+L Switch:SW_Push SW2
 U 1 1 6014049A
 P 15100 4400
-F 0 "SW?" H 15100 4685 50  0000 C CNN
+F 0 "SW2" H 15100 4685 50  0000 C CNN
 F 1 "SW_Push" H 15100 4594 50  0000 C CNN
-F 2 "" H 15100 4600 50  0001 C CNN
+F 2 "Button_Switch_THT:SW_PUSH_6mm" H 15100 4600 50  0001 C CNN
 F 3 "~" H 15100 4600 50  0001 C CNN
 	1    15100 4400
@@
 Connection ~ 14800 4050
 $Comp
-L Switch:SW_Push SW?
+L Switch:SW_Push SW1
 U 1 1 6040825D
 P 15100 3700
-F 0 "SW?" H 15100 3985 50  0000 C CNN
+F 0 "SW1" H 15100 3985 50  0000 C CNN
 F 1 "SW_Push" H 15100 3894 50  0000 C CNN
-F 2 "" H 15100 3900 50  0001 C CNN
+F 2 "Button_Switch_THT:SW_PUSH_6mm" H 15100 3900 50  0001 C CNN
 F 3 "~" H 15100 3900 50  0001 C CNN
 	1    15100 3700
