File: Placa/Placa tesis.kicad_pcb (KiCad board)
At the start: 2 copper layers, 100 x 100 mm, 204 parts, among them J1 Conn_01x03, J10 Conn_01x01, J11 USB_B_Micro, J12 Conn_01x01, J13 Conn_01x05, J14 Conn_01x08, J15 Conn_01x04, J2 Conn_01x04, J3 Conn_01x02, J4 Conn_01x03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

Commit message: actualizacion
Parts:
- removed the BT1 at (147.6, 137.6)
- removed the C1 at (146.2, 93.4)
- removed the C10 at (164.6, 105.9)
- removed the C11 at (101.2, 109.2)
- removed the C12 at (98.8, 109.2)
- removed the C13 at (96.3, 109.2)
- removed the C14 at (88.1, 108.8)
- removed the C15 at (88.2, 96.5)
- removed the C16 at (92.7, 108.8)
- removed the C2 at (146.3, 99.3)
- removed the C3 at (146.3, 102.1)
- removed the C4 at (146.4, 108.5)
- removed the C9 at (161.8, 105.9)
- removed the D5 at (147.7, 132.0)
- removed the J1 at (169.7, 103.8)
- removed the J10 at (147.6, 126.2)
- removed the J11 at (87.1, 102.7)
- removed the J12 at (147.6, 122.3)
- removed the J13 at (162.1, 110.6)
- removed the J14 at (158.4, 103.0)
- removed the J15 at (165.8, 120.7)
- removed the J2 at (107.7, 94.8)
- removed the J3 at (167.6, 96.6)
- removed the J4 at (143.3, 117.4)
- removed the J5 at (135.0, 139.2)
- removed the J6 at (118.6, 95.9)
- removed the J7 at (106.9, 139.5)
- removed the J8 at (84.7, 114.1)
- removed the J9 at (103.9, 99.8)
- removed the OutP at (138.2, 113.7)
- removed the PWR1 at (174.1, 98.5)
- removed the Q1 at (131.4, 129.5)
- removed the Q2 at (131.4, 118.8)
- removed the Q3 at (131.4, 108.1)
- removed the Q4 at (131.4, 97.4)
- removed the R1 at (146.4, 111.2)
- removed the R10 at (142.3, 109.8)
- removed the R11 at (91.9, 100.0)
- removed the R12 at (155.1, 96.5)
- removed the R13 at (171.9, 119.5)
- removed the R14 at (171.9, 121.9)
- removed the R15 at (178.5, 100.2)
- removed the R2 at (146.5, 105.2)
- removed the R24 at (171.7, 98.5)
- removed the R26 at (139.6, 120.5)
- removed the R27 at (139.5, 109.4)
- removed the R28 at (91.9, 104.8)
- removed the R3 at (127.3, 132.4)
- removed the R30 at (100.8, 95.3)
- removed the R31 at (102.7, 105.4)
- removed the R32 at (102.7, 103.0)
- removed the R33 at (95.0, 95.3)
- removed the R34 at (97.9, 95.3)
- removed the R35 at (92.0, 95.3)
- removed the R4 at (127.3, 121.4)
- removed the R5 at (127.3, 110.5)
- removed the R6 at (127.3, 99.7)
- removed the R7 at (141.0, 95.8)
- removed the R8 at (146.1, 95.8)
- removed the R9 at (141.1, 93.4)
- removed the REF** at (110.3, 138.4)
- removed the REF** at (110.3, 113.3)
- removed the REF** at (110.3, 126.7)
- removed the REF** at (110.3, 108.3)
- removed the REF** at (110.3, 118.4)
- removed the REF** at (110.3, 95.0)
- removed the REF** at (110.3, 136.7)
- removed the REF** at (110.3, 125.0)
- removed the REF** at (110.3, 98.3)
- removed the REF** at (110.3, 93.3)
- removed the REF** at (110.3, 121.7)
- removed the REF** at (110.3, 130.0)
- removed the REF** at (110.3, 131.7)
- removed the REF** at (110.3, 128.4)
- removed the REF** at (110.3, 116.7)
- removed the REF** at (110.3, 120.0)
- removed the REF** at (110.3, 110.0)
- removed the REF** at (110.3, 115.0)
- removed the REF** at (110.3, 135.0)
- removed the REF** at (110.3, 91.6)
- removed the REF** at (110.3, 105.0)
- removed the REF** at (110.3, 101.7)
- removed the REF** at (110.3, 133.4)
- removed the REF** at (178.5, 95.5)
- removed the REF** at (115.4, 137.8)
- removed the REF** at (110.3, 103.3)
- removed the REF** at (110.3, 100.0)
- removed the REF** at (110.3, 96.6)
- removed the REF** at (110.3, 106.7)
- removed the REF** at (110.3, 123.4)
- removed the REF** at (110.3, 111.7)
- removed the Rx2 at (105.0, 109.1)
- removed the TH1 at (142.3, 113.9)
- removed the Tx2 at (107.6, 109.1)
- removed the U2 at (165.8, 120.4)
- removed the U3 at (154.8, 104.4)
- removed the U4 at (139.2, 102.1)
- removed the U5 at (165.6, 136.8)
- removed the U6 at (95.8, 136.0)
- removed the U9 at (97.1, 102.4)
- added R16: 10k, Resistor_SMD:R_1206_3216Metric, F.Cu at (77.3, 47.3)
- added R17: 10k, Resistor_SMD:R_1206_3216Metric, F.Cu at (77.3, 52.0)
- added R18: 10k, Resistor_SMD:R_1206_3216Metric, F.Cu at (121.3, 36.3)
- added R19: 10k, Resistor_SMD:R_1206_3216Metric, F.Cu at (116.7, 72.0)
- added SW1: SW_Push, Button_Switch_THT:SW_PUSH_6mm, F.Cu at (72.8, 41.2)
- added SW2: SW_Push, Button_Switch_THT:SW_PUSH_6mm, F.Cu at (124.6, 33.9)
- C1: value 10n -> 1u
- C2, C4: value C -> 1u
- C3: value C -> 2.2n
- R1, R7: value R -> 10k
- R2: value R -> 4.7k
- R8: value R -> 1.5k
Connections:
- U4 pad 29: GND -> (no net)
Routing:
- net (no net): track 1941.2 -> 0.00 mm, vias 76 -> 0
- removed copper zone on B.Cu, net (none)
- removed copper zone on F.Cu, net (none)
Other:
- board size 100 x 100 mm -> 100 x 50 mm

Commit message: La venganza
Parts:
- removed C11: 4.7u, Capacitor_SMD:C_1206_3216Metric
- removed C12, C16: 100n, Capacitor_SMD:C_1206_3216Metric
- removed C13: 10n, Capacitor_SMD:C_1206_3216Metric
- removed C14, C15: 47p, Capacitor_SMD:C_1206_3216Metric
- removed J11: USB_B_Micro, Connector_USB:USB_Micro-B_Wuerth_629105150521
- removed J2: Conn_01x04, Connector_PinHeader_2.54mm:PinHeader_1x04_P2.54mm_Vertical
- removed J7, J8: Conn_01x11, Connector_PinHeader_2.54mm:PinHeader_1x11_P2.54mm_Vertical
- removed J9: Conn_01x03, Connector_PinHeader_2.54mm:PinHeader_1x03_P2.54mm_Vertical
- removed R11, R28: 27, Resistor_SMD:R_1206_3216Metric
- removed R16, R17, R18: 10k, Resistor_SMD:R_1206_3216Metric
- removed R30, R33, R34, R35: 10K, Resistor_SMD:R_1206_3216Metric
- removed R31, R32: 270, Resistor_SMD:R_1206_3216Metric
- removed the REF** at (155.3, 91.2)
- removed the REF** at (155.3, 76.1)
- removed the REF** at (155.3, 74.5)
- removed the REF** at (155.3, 72.8)
- removed the REF** at (155.3, 71.1)
- removed the REF** at (155.3, 67.8)
- removed the REF** at (155.3, 69.5)
- removed the REF** at (155.3, 66.1)
- removed the REF** at (155.3, 64.5)
- removed the REF** at (155.3, 62.8)
- removed the REF** at (155.3, 61.1)
- removed the REF** at (155.3, 89.5)
- removed the REF** at (155.3, 59.4)
- removed the REF** at (155.3, 57.8)
- removed the REF** at (155.3, 56.1)
- removed the REF** at (155.3, 54.4)
- removed the REF** at (155.3, 52.8)
- removed the REF** at (155.3, 51.1)
- removed the REF** at (155.3, 49.4)
- removed the REF** at (155.3, 47.8)
- removed the REF** at (155.3, 46.1)
- removed the REF** at (155.3, 44.4)
- removed the REF** at (155.3, 87.8)
- removed the REF** at (155.3, 86.2)
- removed the REF** at (155.3, 84.5)
- removed the REF** at (155.3, 82.8)
- removed the REF** at (155.3, 81.1)
- removed the REF** at (155.3, 79.5)
- removed the REF** at (155.3, 77.8)
- removed Rx2, Tx2: LED, LED_SMD:LED_1206_3216Metric
- removed SW1, SW2: SW_Push, Button_Switch_THT:SW_PUSH_6mm
- removed U6: ESP-12E, RF_Module:ESP-12E
- removed U9: FT230XS, Package_SO:SSOP-16_3.9x4.9mm_P0.635mm
- J1: value Conn_01x03 -> OKI-78SR
- J13: value Conn_01x05 -> BH1750; moved to B.Cu
- J14: value Conn_01x08 -> INA226; moved to B.Cu
- J15: moved to B.Cu
- J3: value Conn_01x02 -> FUENTE; moved to B.Cu
- J4: value Conn_01x03 -> DHT11
- J5: value Conn_01x04 -> COMM
- moved J3 5.08 mm to (103.1, 86.1), turned to 180 degrees
- turned J13 to 0 degrees
- turned J14 to 0 degrees
- turned J15 to 180 degrees
Connections:
- J3 pad 1: GND -> VinS
- J3 pad 2: VinS -> GND
- R15 pad 2: Net-(R15-Pad2) -> V5
- U2 pad 11: Net-(R15-Pad2) -> V5
- U2 pad 16: Net-(R15-Pad2) -> V5
- U2 pad 25: Net-(R15-Pad2) -> V5
- U5 pad 8: Net-(R15-Pad2) -> V5
Routing:
- net Net-(R15-Pad2): track 88.5 -> 0.00 mm, vias 5 -> 0
- net V5: track 129.5 -> 218.1 mm, vias 4 -> 9
- net Net-(C16-Pad1): track 43.4 -> 0.00 mm
- net Net-(C11-Pad1): track 29.0 -> 0.00 mm, vias 2 -> 0
- net Net-(J2-Pad4): track 16.7 -> 0.00 mm, vias 2 -> 0
- net Net-(J8-Pad1): track 14.9 -> 0.00 mm
- net Net-(J7-Pad11): track 14.9 -> 0.00 mm
- net Net-(J2-Pad3): track 12.8 -> 0.00 mm
- net Net-(J7-Pad10): track 11.8 -> 0.00 mm
- net Net-(J8-Pad2): track 11.4 -> 0.00 mm
- net Net-(C14-Pad1): track 10.3 -> 0.00 mm
- net Net-(C15-Pad1): track 10.2 -> 0.00 mm
- net Net-(J8-Pad3): track 8.10 -> 0.00 mm
- net Net-(J7-Pad9): track 8.10 -> 0.00 mm
- net Net-(R28-Pad1): track 7.73 -> 0.00 mm, vias 2 -> 0
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- removed copper zone on B.Cu, net GND2
- removed copper zone on F.Cu, net GND2
Other:
- board size 100 x 50 mm -> 71.1 x 49.9 mm
